Commit message: 从xacro中找到一年前计算的关节位置的重设

File: dancer_urdf_model/model/dancer_urdf_model.URDF (robot description, URDF)
Before this commit: robot dancer_urdf_model, 22 links, 21 joints
Joints:
- joint joint_arm_left: origin xyz=-0.46902 -0.2921 0.00017561 rpy=-1.5708 -0.59813 1.5708 -> xyz=-0.46902 -0.2921 0.00017561 rpy=-1.5708 1.09187 1.5708
- joint joint_arm_right: origin xyz=-0.25942 -0.2921 0.00017561 rpy=-1.5708 1.0373 1.5708 -> xyz=-0.25942 -0.2921 0.00017561 rpy=-1.5708 1.0973 1.5708
- joint joint_body_hip2_left: origin xyz=0.0493 0.033966 -0.0015267 rpy=3.0498 0.044917 1.5708 -> xyz=0.0493 0.033966 -0.0015267 rpy=3.1698 0.044917 1.5708
- joint joint_body_hip2_right: origin xyz=0.031042 0.015283 0.0465 rpy=1.479 0 0.4575 -> xyz=0.031042 0.015283 0.0465 rpy=2.299 0 0.4575
- joint joint_body_hip_left: origin xyz=0.045 -0.0122 0.065 rpy=1.5708 0 -1.5708 -> xyz=0.045 -0.0122 0.065 rpy=1.6008 0 -1.5708
- joint joint_body_hip_right: origin xyz=-0.045 -0.015 0.065 rpy=1.5708 -1.0684 0 -> xyz=-0.045 -0.015 0.065 rpy=1.5708 -1.1184 0
- joint joint_hand_left: origin xyz=0 -0.136 0.05255 rpy=0.59813 -1.5708 0 -> xyz=0 -0.136 0.05255 rpy=-2.36187 -1.5708 0
- joint joint_hand_right: origin xyz=0 -0.136 0.00845 rpy=2.1043 1.5708 0 -> xyz=0 -0.136 0.00845 rpy=-0.6557 1.5708 0
- joint joint_leg2_left: origin xyz=-0.0006 0.098703 -0.068248 rpy=0 0 0 -> xyz=-0.0006 0.098703 -0.068248 rpy=-1.05 0 0
- joint joint_leg2_right: origin xyz=-0.0016 -0.020351 -0.11826 rpy=0 0 0 -> xyz=-0.0016 -0.020351 -0.11826 rpy=0.94 0 0
- joint joint_leg3_left: origin xyz=0.0006 0.11852 0.05341 rpy=0 0 0 -> xyz=0.0006 0.11852 0.05341 rpy=0.41 0 0
- joint joint_leg3_right: origin xyz=0 -0.1146 -0.061382 rpy=0 0 0 -> xyz=0 -0.1146 -0.061382 rpy=-1.05 0 0
- joint joint_leg4_left: origin xyz=-0.0241 -0.0065502 0.035907 rpy=-2.9765 -0.0732 0.41369 -> xyz=-0.0241 -0.0065502 0.035907 rpy=-2.9765 -0.0132 0.03369
- joint joint_leg4_right: origin xyz=-0.0265 -0.035971 0.0061902 rpy=1.883 -0.9859 2.8787 -> xyz=-0.0265 -0.035971 0.0061902 rpy=1.753 0.0141 3.1487
- joint joint_leg_left: origin xyz=-0.034 0.0013682 0.024061 rpy=-2.6864 -1.514 1.5708 -> xyz=-0.034 0.0013682 0.024061 rpy=-1.0064 -1.514 1.5708
- joint joint_leg_right: origin xyz=-0.0346 -0.019079 -0.02063 rpy=-0.34551 0.82443 -1.5708 -> xyz=-0.0346 -0.019079 -0.02063 rpy=0.20449 0.82443 -1.5708

Commit message: bullet不需要世界坐标系,加上反而会导致action错误

File: dancer_urdf_model/model/dancer_urdf_model.URDF (robot description, URDF)
Before this commit: robot dancer_urdf_model, 22 links, 21 joints
Links:
- removed link world_link
Joints:
- removed joint joint_world

Commit message: urdf文件修复完成

File: dancer_urdf_model/model/dancer_urdf_model.URDF (robot description, URDF)
Before this commit: robot dancer_urdf_model, 21 links, 20 joints
Links:
- removed link body_camera
- removed link body_hip
- removed link leg3_left
- removed link leg3_right
- removed link leg4_left
- removed link leg4_right
- added link foot1_left, mass 0.158402372500407; collision mesh filename=package://dancer_urdf_model/meshes/foot1_left.STL; visual mesh filename=package://dancer_urdf_model/meshes/foot1_left.STL
- added link foot1_right, mass 0.158402372500407; collision mesh filename=package://dancer_urdf_model/meshes/foot1_right.STL; visual mesh filename=package://dancer_urdf_model/meshes/foot1_right.STL
- added link foot2_left, mass 0.14417666873715; collision mesh filename=package://dancer_urdf_model/meshes/foot2_left.STL; visual mesh filename=package://dancer_urdf_model/meshes/foot2_left.STL
- added link foot2_right, mass 0.143428639592448; collision mesh filename=package://dancer_urdf_model/meshes/foot2_right.STL; visual mesh filename=package://dancer_urdf_model/meshes/foot2_right.STL
- link arm_left: mass 0.142976459032186 -> 0.140880460038681
- link arm_right: mass 0.141656759847187 -> 0.140880462107965
- link body_chest: mass 0.66907 -> 0.882484739618511
- link body_head: mass 0.0560380421735799 -> 0.05496
- link body_head2: mass 0.067365 -> 0.0803703275300652
- link body_hip2_left: mass 0.178226116015845 -> 0.159177872474359
- link body_hip2_right: mass 0.178226118022815 -> 0.159177872474359
- link body_hip_left: mass 0.0513468076618724 -> 0.0606904859381705
- link body_hip_right: mass 0.0513468076618724 -> 0.0606904859337575
- link hand_left: mass 0.021948273112724 -> 0.0240442691962686
- link hand_right: mass 0.021948273112724 -> 0.0227245679584811
- link leg2_left: mass 0.0278306854029525 -> 0.0468789275178147
- link leg2_right: mass 0.0278306854029525 -> 0.0468789275178147
- link leg_left: mass 0.117898503490257 -> 0.11789850487658
- link leg_right: mass 0.117898502766572 -> 0.11789850487658
Joints:
- removed joint joint_body_camera
- removed joint joint_body_hip
- removed joint joint_leg3_left
- removed joint joint_leg3_right
- removed joint joint_leg4_left
- removed joint joint_leg4_right
- added joint joint_foot1_left: type continuous, parent leg2_left, child foot1_left, origin xyz=-0.0102535550345806 0.0220306418254577 -0.128119673824045 rpy=0 0 0, axis 1 0 0
- added joint joint_foot1_right: type continuous, parent leg2_right, child foot1_right, origin xyz=0 0.011730641825261 -0.129469656840417 rpy=0 0 0, axis 1 0 0
- added joint joint_foot2_left: type continuous, parent foot1_left, child foot2_left, origin xyz=0.522711919869236 -0.21233840256255 0.200834517315037 rpy=0 0 0, axis 0 1 0
- added joint joint_foot2_right: type continuous, parent foot1_right, child foot2_right, origin xyz=-0.0385989383789022 0 0 rpy=0 0 0, axis 0 1 0
- joint joint_arm_left: axis 0 0 1 -> 0.999887496502133 0 -0.0149998112887317; origin xyz=-0.46902 -0.2921 0.00017561 rpy=-1.5708 1.09187 1.5708 -> xyz=-0.480637621395787 -0.270857071736484 0.200567760736966 rpy=1.5707963267949 0 0
- joint joint_arm_right: axis 0 0 1 -> 0.999887496502132 0 -0.0149998112887528; origin xyz=-0.25942 -0.2921 0.00017561 rpy=-1.5708 1.0973 1.5708 -> xyz=-0.690210517946081 -0.274000979336581 0.20056776073696 rpy=1.5707963267949 0 0
- joint joint_body_head: axis 0 1 0 -> 0.0149998112887428 0 0.999887496502132; origin xyz=-0.39482 -0.32209 -0.014452 rpy=2.6872 -0.050522 -3.1169 -> xyz=-0.615612428513425 -0.285967486211966 0.20056776073696 rpy=1.5707963267949 0 0
- joint joint_body_head2: axis -1 0 0 -> 0.999887496502133 0 -0.0149998112887384; origin xyz=0.02015 -0.031182 0 rpy=-1.1164 0 0 -> xyz=0.0507513535336471 0 0.0497102139820205 rpy=0 0 0
- joint joint_body_hip2_left: axis -1 0 0 -> 0 1 0; origin xyz=0.0493 0.033966 -0.0015267 rpy=3.1698 0.044917 1.5708 -> xyz=0.000579999589308322 0 0.038662775562355 rpy=0 0 0
- joint joint_body_hip2_right: axis -1 0 0 -> 0 1 0; origin xyz=0.031042 0.015283 0.0465 rpy=2.299 0 0.4575 -> xyz=0.000542083800765036 0 0.0361353089051728 rpy=0 0 0
- joint joint_body_hip_left: axis -1 0 0 -> 0.0149998112887428 0 0.999887496502133; origin xyz=0.045 -0.0122 0.065 rpy=1.6008 0 -1.5708 -> xyz=-0.574767957608413 -0.00862238094696859 0.200607760736968 rpy=1.5707963267949 0 0; parent body_hip -> body_chest
- joint joint_body_hip_right: axis 0 0 1 -> 0.0149998112887428 0 0.999887496502133; origin xyz=-0.045 -0.015 0.065 rpy=1.5708 -1.1184 0 -> xyz=-0.664719916505049 -0.0124998306201608 0.20060776073697 rpy=1.5707963267949 0 0; parent body_hip -> body_chest
- joint joint_hand_left: axis 1 0 0 -> 0.999887496502131 0 -0.0149998112888278; origin xyz=0 -0.136 0.05255 rpy=-2.36187 -1.5708 0 -> xyz=-0.00831303371965708 0 -0.135890594230151 rpy=0 0 0
- joint joint_hand_right: axis 1 0 0 -> 0.999887496502134 0 -0.0149998112886474; origin xyz=0 -0.136 0.00845 rpy=-0.6557 1.5708 0 -> xyz=-0.0493202167072464 0 -0.135275425015181 rpy=0 0 0
- joint joint_leg2_left: axis -1 0 0 -> 1 0 0; origin xyz=-0.0006 0.098703 -0.068248 rpy=-1.05 0 0 -> xyz=0.0499806689582331 0 -0.120000000000317 rpy=0 0 0
- joint joint_leg2_right: origin xyz=-0.0016 -0.020351 -0.11826 rpy=0.94 0 0 -> xyz=0.0513478626051265 0 -0.120000000000008 rpy=0 0 0
- joint joint_leg_left: axis -1 0 0 -> 1 0 0; origin xyz=-0.034 0.0013682 0.024061 rpy=-1.0064 -1.514 1.5708 -> xyz=0.0117489242262162 -0.0103000000000123 0 rpy=0 0 0
- joint joint_leg_right: origin xyz=-0.0346 -0.019079 -0.02063 rpy=0.20449 0.82443 -1.5708 -> xyz=-0.0127489242262093 0 0 rpy=0 0 0

Commit message: 修复模型左脚坐标系

File: dancer_urdf_model/model/dancer_urdf_model.URDF (robot description, URDF)
Before this commit: robot dancer_urdf_model, 19 links, 18 joints
Joints:
- joint joint_foot2_left: origin xyz=0.522711919869236 -0.21233840256255 0.200834517315037 rpy=0 0 0 -> xyz=-0.0530760381498626 -0.031751075773801 0 rpy=0 0 0

Commit message: 修改动作和重力和质量之后终于成功爬起

File: dancer_urdf_model/model/dancer_urdf_model.URDF (robot description, URDF)
Before this commit: robot dancer_urdf_model, 19 links, 18 joints
Links:
- link body_chest: mass 0.882484739618511 -> 0.088248473961851
